Commit message: new changes

File: src/simple2wheeler/urdf/simple2wheeler.xacro (robot description, xacro)
@@ -95,4 +95,35 @@
             <joint_properties damping="1.0" friction="1.0"/>
         </joint>
+        <link name="camera_link">
+            <collision>
+            </collision>
+            <visual>
+            </visual>
+        </link>
+        <joint name="camera_joint" type="fixed">
+            <origin rpy="0 0 0" xyz="0.25 0.07 0.07"/>
+            <child link="camera_link"/>
+            <parent link="link_chassis"/>
+        </joint>
+        <gazebo reference="camera_link">
+            <sensor type="camera" name="camera_sensor">
+                <update_rate>30</update_rate>
+                <camera>
+                    <horizontal_fov>1.34</horizontal_fov>
+                    <image>
+                        <format>R8G8B8</format>
+                        <width>1020</width>
+                        <height>1020</height>
+                    </image>
+                    <clip>
+                        <near>0.01</near>
+                        <far>30</far>
+                    </clip>
+                </camera>
+                <plugin name="camera_controller" filename="libgazebo_ros_camera.so">
+                    <alwaysOn>true</alwaysOn>
+                    <updateRate>30.0</updateRate>
+                    <cameraName>/camera</cameraName>
+                    <CameraTopicName>image_raw</CameraTopicName>
         <gazebo>
             <plugin filename="libgazebo_ros_diff_drive.so" name="differential_drive_controller">

Commit message: new things

File: src/simple2wheeler/urdf/simple2wheeler.xacro (robot description, xacro)
@@ -125,8 +125,50 @@
                     <updateRate>30.0</updateRate>
                     <cameraName>/camera</cameraName>
-                    <CameraTopicName>image_raw</CameraTopicName>
+                    <imageTopicName>image_raw</imageTopicName>
+                    <cameraInfoTopicName>camera_info</cameraInfoTopicName>
+                    <frameName>camera_link</frameName>
+                    <hackBaseLine>0.07</hackBaseLine>
+                    <distortionK1>0</distortionK1>
+                    <distortionK2>0</distortionK2>
+                    <distortionK3>0</distortionK3>
+                    <distortionT1>0</distortionT1>
+                    <distortionT2>0</distortionT2>
+                </plugin>
+            </sensor>
+        </gazebo>
+        <link name="imu_link">
+            <collision>
+            </collision>
+            <visual>
+            </visual>
+        </link>
+        <joint name="imu_joint" type="fixed">
+            <origin rpy="0 0 0" xyz="0.0 0.0 0.07"/>
+            <child link="imu_link"/>
+            <parent link="link_chassis"/>
+        </joint>
+        <gazebo reference="imu_link">
+            <gravity>true</gravity>
+            <sensor name="imu_sensor" type="imu">
+                <alwaysOn>true</alwaysOn>
+                <update_rate>10</update_rate>
+                <visualize>true</visualize>
+                <topic>_default_topic_</topic>
+                <plugin filename="libgazebo_ros_imu_sensor.so" name="imu_plugin">
+                    <topicName>imu</topicName>
+                    <bodyName>imu_link</bodyName>
+                    <updateRateHZ>10</updateRateHZ>
+                    <gaussianNoise>0.0</gaussianNoise>
+                    <xyzOffset>0 0 0 </xyzOffset>
+                    <rpyOffset>0 0 0 </rpyOffset>
+                    <frameName>imu_link</frameName>
+                    <inertialOrientationAsReference>false</inertialOrientationAsReference>
+                </plugin>
+                <pose> 0 0 0 0 0 0 </pose>
+            </sensor>
+        </gazebo>
         <gazebo>
             <plugin filename="libgazebo_ros_diff_drive.so" name="differential_drive_controller">
-                <lecacyMode>false</lecacyMode>
+                <legacyMode>false</legacyMode>
                 <alwaysOn>true</alwaysOn>
                 <updateRate>20</updateRate>

Commit message: updated

File: src/simple2wheeler/urdf/simple2wheeler.xacro (robot description, xacro)
@@ -184,3 +184,57 @@
             </plugin>
         </gazebo>
+        <link name="lidar_link">
+            <visual>
+                <geometry>
+                    <mesh filename="package://simple2wheeler/meshes/rplidar_a2_simple.stl" />
+                </geometry>
+            </visual>
+            <collision>
+                <geometry>
+                    <mesh filename="package://simple2wheeler/meshes/rplidar_a2_simple.stl" />
+                </geometry>
+            </collision>
+            <inertial>
+                <mass value="0.125"/>
+                <origin xyz="0 0 -0.026" />
+                <inertia ixx="0.000144185" ixy="0.0" ixz="0.0"
+                    iyy="0.00144185" iyz="0.0"
+                    izz="0.00144185" />
+            </inertial>
+        </link>
+        <joint name="lidar_joint" type="fixed">
+            <parent link="link_chassis" />
+            <child link="lidar_link" />
+            <origin rpy="0 0 0" xyz="0 0 0.17" />
+        </joint>
+        <gazebo reference="lidar_link">
+            <sensor type="ray" name="lidar">
+                <alwaysOn>true</alwaysOn>
+                <update_rate>10</update_rate>
+                <pose> 0 0 0 0 0 0 </pose>
+                <visualize>true</visualize>
+                <ray>
+                    <scan>
+                        <horizontal>
+                            <samples>400</samples>
+                            <resolution>0.9</resolution>
+                            <min_angle>-3.142</min_angle>
+                            <max_angle>3.142</max_angle>
+                        </horizontal>
+                    </scan>
+                    <range>
+                        <min>0.15</min>
+                        <max>6</max>
+                        <resolution>0.01</resolution>
+                    </range>
+                </ray>
+                <plugin name="gazebo_ros_lidar_controller" filename="libgazebo_ros_laser.so">
+                    <gaussianNoise>0.005</gaussianNoise>
+                    <alwaysOn>true</alwaysOn>
+                    <updateRate>10</updateRate>
+                    <topicName>lidar</topicName> <!--/lidar should work also-->
+                    <frameName>lidar_link</frameName>
+                </plugin>
+            </sensor>
+        </gazebo>
     </robot>

Commit message: more changes

File: src/simple2wheeler/urdf/simple2wheeler.xacro (robot description, xacro)
@@ -206,5 +206,5 @@
             <parent link="link_chassis" />
             <child link="lidar_link" />
-            <origin rpy="0 0 0" xyz="0 0 0.17" />
+            <origin rpy="0 0 0" xyz="0 0 0.07" />
         </joint>
         <gazebo reference="lidar_link">
